File: currentsource/linearsource_mod/linearsource_mod.kicad_pcb (KiCad board)
At the start: 2 copper layers, 45.7 x 22.2 mm, 18 parts, among them P1 CONN_01X05, P2 CONN_01X04, Q1 PSMN017-30BL, Q2 BC849, U1 LM358

Commit message: currentsource: Commit changes
Parts:
- removed TP1: TEST, SMD_Packages:1Pin
- Q1: value PSMN017-30BL -> Q_NMOS_GDS; footprint TO_SOT_Packages_SMD:TO-263-3Lead -> Edge:TO-220_Horizontal
- moved R5 5.12 mm to (178.8, 83.2), turned to 180 degrees
- moved Q1 4.02 mm to (182.6, 73.1)
- moved R4 2.69 mm to (177.5, 72.4), turned to 180 degrees
- moved P2 2.54 mm to (180.7, 87.7)
Connections:
- Q1 pad 1: I_out- -> Net-(Q1-Pad1)
- Q1 pad 2: Net-(Q1-Pad2) -> I_out-
- R4 pad 1: Net-(Q1-Pad2) -> Net-(Q1-Pad1)
Routing:
- net I_out-: track 36.5 -> 0.00 mm
- net I_sense: track 32.9 -> 10.7 mm
- net Net-(Q1-Pad2): track 17.0 -> 0.00 mm
- net GND: track 90.4 -> 84.8 mm
- net Net-(R4-Pad2): track 4.27 -> 0.00 mm
- net (no net): track 0.00 -> 0.63 mm
