File: guitar-effects/peq10/peq10.kicad_sch (KiCad schematic)
At the start: 20 parts, among them J1 Conn_01x04, J2 Conn_01x04, U1 4052, U2 NE5532, U3 NE5532, U4 NE5532, U5 PCF8574

Commit message: guitar-effects: Notes on parametric EQ
Connections:
- net GND: now also U1.7 (VEE), U1.8 (VSS), U5.8 (VSS)
- net VDD: now also U5.16 (VDD)
- net VSS: now also U1.16 (VDD)
- net at U5.10 (P5): no longer U1.5 (Y1)
- net at U5.11 (P6): no longer U1.2 (Y2)
- net at U5.12 (P7): no longer U1.4 (Y3)
- net at U5.4 (P0): now also U1.6 (Inh); no longer U1.12 (X0)
- net at U5.5 (P1): now also U1.10 (A); no longer U1.14 (X1)
- net at U5.6 (P2): now also U1.9 (B); no longer U1.15 (X2)
- net at U5.7 (P3): no longer U1.11 (X3)
- net at U5.9 (P4): no longer U1.1 (Y0)
- net MUX: now reaches U1.13 (X)
Other:
- note added: "FIXME: use virtual ground"
- note added: "TODO: add cut/boost"
- moved on the sheet: U1, U4A, U5
